Commit message: 仿真新增tof和3D lidar

File: robot_description/urdf/four_wheel_steering_robot.urdf (robot description, URDF)
Before this commit: robot /home/CNF2025495045/workspace/nav_for_4WS/src/robot_webots_sim/worlds/four_wheel_steering_robot.urdf, 13 links, 12 joints
Links:
- removed link inertial unit
- added link imu
- added link lidar
- added link tof
Joints:
- removed joint base_link_inertial unit_joint
- added joint base_link_imu_joint: type fixed, parent base_link, child imu, origin xyz=0 0 0 rpy=0 0 0
- added joint base_link_lidar_joint: type fixed, parent base_link, child lidar, origin xyz=0.2 0 0.06 rpy=0 0.523595 0
- added joint base_link_tof_joint: type fixed, parent base_link, child tof, origin xyz=0.218435 0 0.031895 rpy=0 -0.261795 0

Commit message: 3D雷达和tof的rviz显示正常

File: robot_description/urdf/four_wheel_steering_robot.urdf (robot description, URDF)
Before this commit: robot /home/CNF2025495045/workspace/nav_for_4WS/src/robot_webots_sim/worlds/four_wheel_steering_robot.urdf, 15 links, 14 joints
Links:
- added link lidar_optical
- added link tof_optical
Joints:
- added joint lidar_to_optical_joint: type fixed, parent lidar, child lidar_optical, origin xyz=0 0 0 rpy=0 0 0
- added joint tof_to_optical_joint: type fixed, parent tof, child tof_optical, origin xyz=0 0 0 rpy=1.570796 3.141592 1.570796
- joint base_link_lidar_joint: origin xyz=0.2 0 0.06 rpy=0 0.523595 0 -> xyz=0.2 0 0.06 rpy=0 0 0

Commit message: 完善webots的imu和lidar

File: robot_description/urdf/four_wheel_steering_robot.urdf (robot description, URDF)
Before this commit: robot /home/CNF2025495045/workspace/nav_for_4WS/src/robot_webots_sim/worlds/four_wheel_steering_robot.urdf, 17 links, 16 joints
Links:
- removed link lidar_optical
- added link accelerometer
- added link gyro
Joints:
- removed joint lidar_to_optical_joint
- added joint base_link_accelerometer_joint: type fixed, parent base_link, child accelerometer, origin xyz=0 0 0 rpy=0 0 0
- added joint base_link_gyro_joint: type fixed, parent base_link, child gyro, origin xyz=0 0 0 rpy=0 0 0
- joint base_link_lidar_joint: origin xyz=0.2 0 0.06 rpy=0 0 0 -> xyz=0 0 0.05 rpy=0 0 0

Commit message: 使用2Dslam，并调整基础导航效果完成

File: robot_description/urdf/four_wheel_steering_robot.urdf (robot description, URDF)
Before this commit: robot /home/CNF2025495045/workspace/nav_for_4WS/src/robot_webots_sim/worlds/four_wheel_steering_robot.urdf, 18 links, 17 joints
Joints:
- joint base_footprint_joint: origin xyz=0 0 0.05 rpy=0 0 0 -> xyz=0 0 0.0 rpy=0 0 0
